Commit message: updated reference doc

File: urdf/x_drive.urdf.xacro (robot description, xacro)
@@ -9,7 +9,7 @@
 	<xacro:property name="wheel_rad" value="0.01375"/>
 	<!-- Stand in link for the world-->
-	<link name='world'/>
+	<link name='base_footprint'/>
 	<!--Chassis link-->
-	<link name="chassis">
+	<link name="base_link">
 		<visual>
 			<geometry>
@@ -79,20 +79,20 @@
 	<joint name="world_2_chassis" type='fixed'>
 		<origin xyz="0 0 0.025" rpy="0 0 0"/>
-		<parent link='world'/>
-		<child link='chassis'/>
+		<parent link='base_footprint'/>
+		<child link='base_link'/>
 	</joint>
 	<joint name="chassis_to_wheel_a" type="continuous">
         <origin xyz="-${wheel_offs} ${wheel_offs} ${wheel_rad}" rpy="0 0 ${pi_4}"/>
-        <parent link="chassis"/>
+        <parent link="base_link"/>
         <child link="wheel_a"/>
     </joint>
 	<joint name="chassis_to_wheel_b" type="continuous">
         <origin xyz="${wheel_offs} -${wheel_offs} ${wheel_rad}" rpy="0 0 ${pi_4}"/>
-        <parent link="chassis"/>
+        <parent link="base_link"/>
         <child link="wheel_b"/>
     </joint>
 	<joint name="chassis_to_wheel_c" type="continuous">
         <origin xyz="${wheel_offs} ${wheel_offs} ${wheel_rad}" rpy="0 0 -${pi_4}"/>
-        <parent link="chassis"/>
+        <parent link="base_link"/>
         <child link="wheel_c"/>
     </joint>

Commit message: it builds!

File: urdf/x_drive.urdf.xacro (robot description, xacro)
@@ -99,6 +99,39 @@
 	<joint name="chassis_to_wheel_d" type="continuous">
         <origin xyz="-${wheel_offs} -${wheel_offs} ${wheel_rad}" rpy="0 0 -${pi_4}"/>
-        <parent link="chassis"/>
+        <parent link="base_link"/>
         <child link="wheel_d"/>
     </joint>
+	<ros2_control name="x_drive_controller" type="system">
+	    <hardware>
+            <plugin>mock_components/GenericSystem</plugin>
+            <param name="mock_sensor_commands">false</param>
+            <param name="state_following_offset">0.0</param>
+        </hardware>
+		<joint name="chassis_to_wheel_a">
+   			<command_interface name="velocity"/>
+			<state_interface name="velocity"/>
+   			<state_interface name="position"/>
+ 		</joint>
+		<joint name="chassis_to_wheel_b">
+   			<command_interface name="velocity"/>
+			<state_interface name="velocity"/>
+   			<state_interface name="position"/>
+ 		</joint>
+		<joint name="chassis_to_wheel_c">
+   			<command_interface name="velocity"/>
+			<state_interface name="velocity"/>
+   			<state_interface name="position"/>
+ 		</joint>
+		<joint name="chassis_to_wheel_d">
+   			<command_interface name="velocity"/>
+			<state_interface name="velocity"/>
+   			<state_interface name="position"/>
+ 		</joint>
+	</ros2_control>
+	<gazebo>
+  		<plugin filename="libgz_ros2_control-system.so" name="gz_ros2_control::GazeboSimROS2ControlPlugin">
+    		<parameters>package://vex_robot/config/omni_wheel_params.yaml</parameters>
+			<controller_manager_prefix_node_name>controller_manager</controller_manager_prefix_node_name>
+  		</plugin>
+	</gazebo>
 </robot>
