Commit message: added sdf file

File: robot_description/models/x_drive/x_drive.urdf.xacro (robot description, xacro)
@@ -2,5 +2,4 @@
 <robot name="x_drive" xmlns:xacro="http://www.ros.org/wiki/xacro">
 	<!-- properties-->
-	<xacro:property name="stl_path" value="package://robot_description/models"/>
 	<xacro:property name="pi_4" value="0.7854"/>
 	<xacro:property name="pi_2" value="1.5708"/>
@@ -14,10 +13,10 @@
 		<visual>
 			<geometry>
-				<mesh filename='${stl_path}/chassis.dae'/>
+				<mesh filename='package://robot_description/models/x_drive/meshes/chassis.dae'/>
 			</geometry>
 		</visual>
 		<collision>
 			<geometry>
-				<mesh filename='package://robot_description/models/chassis.dae'/>
+				<mesh filename='package://robot_description/models/x_drive/meshes/chassis.dae'/>
 			</geometry>
 			<material name="pink">
@@ -28,15 +27,12 @@
             <origin xyz="0 0 0" rpy="0 0 0"/>
             <mass value="8.789"/>
-            <inertia
-                ixx="144.802"
-				ixy="0"
-				ixz="0"
-				iyx="0"
-                iyy="144.802"
-				iyz="0"
-				izx="0"
-				izy="0"
-                izz="288.141"/>
-        </inertial>
+           <inertia
+      			ixx="0.01"
+				ixy="0.0"
+				ixz="0.0"
+				iyy="0.01"
+				iyz="0.0"
+				izz="0.01"/>
+    </inertia>
 	</link>
 	<!-- wheels -->
@@ -45,5 +41,5 @@
 			<visual>
 				<geometry>
-					<mesh filename='package://robot_description/models/wheel.stl'/>
+					<mesh filename='package://robot_description/models/x_drive/meshes/wheel.dae'/>
 				</geometry>
 				<material name="dark_grey">
@@ -53,5 +49,5 @@
 			<collision>
 				<geometry>
-					<mesh filename='package://robot_description/models/wheel.stl'/>
+					<mesh filename='package://robot_description/models/x_drive/meshes/wheel.dae'/>
 				</geometry>
 			</collision>
@@ -60,13 +56,10 @@
             	<mass value="0.076"/>
 				<inertia
-					ixx="0.055"
-					ixy="0"
-					ixz="0"
-					iyx="0"
-					iyy="0.0988"
-					iyz="0"
-					izx="0"
-					izy="0"
-					izz="0.055"/>
+      			ixx="0.01"
+				ixy="0.0"
+				ixz="0.0"
+				iyy="0.01"
+				iyz="0.0"
+				izz="0.01"/>
         	</inertial>
 		</link>

Commit message: various bug fixes

File: robot_description/models/x_drive/x_drive.urdf.xacro (robot description, xacro)
@@ -34,5 +34,5 @@
 				iyz="0.0"
 				izz="0.01"/>
-    </inertia>
+    		</inertial>
 	</link>
 	<!-- wheels -->

File: robot_gazebo/models/x_drive.urdf.xacro (robot description, xacro)
@@ -2,5 +2,4 @@
 <robot name="x_drive" xmlns:xacro="http://www.ros.org/wiki/xacro">
 	<!-- properties-->
-	<xacro:property name="stl_path" value="package://vex_robot/models"/>
 	<xacro:property name="pi_4" value="0.7854"/>
 	<xacro:property name="pi_2" value="1.5708"/>
@@ -9,15 +8,15 @@
 	<xacro:property name="wheel_rad" value="0.01375"/>
 	<!--world link-->
-	<link name='base_footprint'/>
+	<link name='world'/>
 	<!--chassis link-->
 	<link name="base_link">
 		<visual>
 			<geometry>
-				<mesh filename='${stl_path}/chassis.dae'/>
+				<mesh filename='package://robot_description/models/x_drive/meshes/chassis.dae'/>
 			</geometry>
 		</visual>
 		<collision>
 			<geometry>
-				<mesh filename='package://robot_description/models/chassis.dae'/>
+				<mesh filename='package://robot_description/models/x_drive/meshes/chassis.dae'/>
 			</geometry>
 			<material name="pink">
@@ -28,15 +27,12 @@
             <origin xyz="0 0 0" rpy="0 0 0"/>
             <mass value="8.789"/>
-            <inertia
-                ixx="144.802"
-				ixy="0"
-				ixz="0"
-				iyx="0"
-                iyy="144.802"
-				iyz="0"
-				izx="0"
-				izy="0"
-                izz="288.141"/>
-        </inertial>
+           <inertia
+      			ixx="0.01"
+				ixy="0.0"
+				ixz="0.0"
+				iyy="0.01"
+				iyz="0.0"
+				izz="0.01"/>
+    		</inertial>
 	</link>
 	<!-- wheels -->
@@ -45,5 +41,5 @@
 			<visual>
 				<geometry>
-					<mesh filename='package://robot_description/models/wheel.stl'/>
+					<mesh filename='package://robot_description/models/x_drive/meshes/wheel.dae'/>
 				</geometry>
 				<material name="dark_grey">
@@ -53,5 +49,5 @@
 			<collision>
 				<geometry>
-					<mesh filename='package://robot_description/models/wheel.stl'/>
+					<mesh filename='package://robot_description/models/x_drive/meshes/wheel.dae'/>
 				</geometry>
 			</collision>
@@ -60,13 +56,10 @@
             	<mass value="0.076"/>
 				<inertia
-					ixx="0.055"
-					ixy="0"
-					ixz="0"
-					iyx="0"
-					iyy="0.0988"
-					iyz="0"
-					izx="0"
-					izy="0"
-					izz="0.055"/>
+      			ixx="0.01"
+				ixy="0.0"
+				ixz="0.0"
+				iyy="0.01"
+				iyz="0.0"
+				izz="0.01"/>
         	</inertial>
 		</link>
@@ -129,3 +122,9 @@
  		</joint>
 	</ros2_control>
+	<gazebo>
+  		<plugin filename="ros2_control-system.so" name="gz_ros2_control::GazeboSimROS2ControlPlugin">
+    		<parameters>package://vex_robot/config/omni_wheel_params.yaml</parameters>
+			<controller_manager_prefix_node_name>controller_manager</controller_manager_prefix_node_name>
+  		</plugin>
+	</gazebo>
 </robot>
