Commit message: converted xacro --> urdf, still crashes

File: robot_gazebo/models/x_drive.urdf.xacro (robot description, xacro)
@@ -1,4 +1,4 @@
 <?xml version='1.0'?>
-<model name="x_drive" xmlns:xacro="http://www.ros.org/wiki/xacro">
+<robot name="x_drive" xmlns:xacro="http://www.ros.org/wiki/xacro">
 	<!-- properties-->
 	<xacro:property name="stl_path" value="package://vex_robot/models"/>
@@ -19,5 +19,5 @@
 		<collision>
 			<geometry>
-				<mesh filename='package://vex_robot/models/chassis.dae'/>
+				<mesh filename='package://robot_description/models/chassis.dae'/>
 			</geometry>
 			<material name="pink">
@@ -45,5 +45,5 @@
 			<visual>
 				<geometry>
-					<mesh filename='package://vex_robot/models/wheel.stl'/>
+					<mesh filename='package://robot_description/models/wheel.stl'/>
 				</geometry>
 				<material name="dark_grey">
@@ -53,5 +53,5 @@
 			<collision>
 				<geometry>
-					<mesh filename='package://vex_robot/models/wheel.stl'/>
+					<mesh filename='package://robot_description/models/wheel.stl'/>
 				</geometry>
 			</collision>
@@ -79,5 +79,5 @@
 	<joint name="world_2_chassis" type='fixed'>
 		<origin xyz="0 0 0.025" rpy="0 0 0"/>
-		<parent link='base_footprint'/>
+		<parent link='world'/>
 		<child link='base_link'/>
 	</joint>
@@ -102,5 +102,5 @@
         <child link="wheel_d"/>
     </joint>
-	<ros2_control name="GazeboSimSystem" type="system">
+	<ros2_control name="x_drive_controller" type="system">
 	    <hardware>
             <plugin>mock_components/GenericSystem</plugin>
@@ -129,9 +129,3 @@
  		</joint>
 	</ros2_control>
-	<gazebo>
-  		<plugin filename="ros2_control-system.so" name="gz_ros2_control::GazeboSimROS2ControlPlugin">
-    		<parameters>package://vex_robot/config/omni_wheel_params.yaml</parameters>
-			<controller_manager_prefix_node_name>controller_manager</controller_manager_prefix_node_name>
-  		</plugin>
-	</gazebo>
-</model>
+</robot>

Commit message: finally, a different error message

File: robot_gazebo/models/x_drive.urdf.xacro (robot description, xacro)
@@ -1,6 +1,7 @@
 <?xml version='1.0'?>
-<model name="x_drive" xmlns:xacro="http://www.ros.org/wiki/xacro">
+<robot name="x_drive" xmlns:xacro="http://www.ros.org/wiki/xacro" xmlns:gz="http://gazebosim.org/schema">
 	<!-- properties-->
-	<xacro:property name="stl_path" value="package://vex_robot/models"/>
+	<xacro:property name="model_path" value="package://robot_description/models"/>
+	<xacro:property name="package_path" value="package://robot_gazebo/config"/>
 	<xacro:property name="pi_4" value="0.7854"/>
 	<xacro:property name="pi_2" value="1.5708"/>
@@ -9,15 +10,15 @@
 	<xacro:property name="wheel_rad" value="0.01375"/>
 	<!--world link-->
-	<link name='base_footprint'/>
+	<link name='world'/>
 	<!--chassis link-->
 	<link name="base_link">
 		<visual>
 			<geometry>
-				<mesh filename='${stl_path}/chassis.dae'/>
+				<mesh filename='${model_path}/chassis.dae'/>
 			</geometry>
 		</visual>
 		<collision>
 			<geometry>
-				<mesh filename='package://vex_robot/models/chassis.dae'/>
+				<mesh filename='${model_path}/chassis.dae'/>
 			</geometry>
 			<material name="pink">
@@ -28,15 +29,12 @@
             <origin xyz="0 0 0" rpy="0 0 0"/>
             <mass value="8.789"/>
-            <inertia
-                ixx="144.802"
-				ixy="0"
-				ixz="0"
-				iyx="0"
-                iyy="144.802"
-				iyz="0"
-				izx="0"
-				izy="0"
-                izz="288.141"/>
-        </inertial>
+           <inertia
+      			ixx="0.01"
+				ixy="0.0"
+				ixz="0.0"
+				iyy="0.01"
+				iyz="0.0"
+				izz="0.01"/>
+    		</inertial>
 	</link>
 	<!-- wheels -->
@@ -45,5 +43,5 @@
 			<visual>
 				<geometry>
-					<mesh filename='package://vex_robot/models/wheel.stl'/>
+					<mesh filename='${model_path}/wheel.dae'/>
 				</geometry>
 				<material name="dark_grey">
@@ -53,5 +51,5 @@
 			<collision>
 				<geometry>
-					<mesh filename='package://vex_robot/models/wheel.stl'/>
+					<mesh filename='${model_path}/wheel.dae'/>
 				</geometry>
 			</collision>
@@ -60,13 +58,10 @@
             	<mass value="0.076"/>
 				<inertia
-					ixx="0.055"
-					ixy="0"
-					ixz="0"
-					iyx="0"
-					iyy="0.0988"
-					iyz="0"
-					izx="0"
-					izy="0"
-					izz="0.055"/>
+      			ixx="0.01"
+				ixy="0.0"
+				ixz="0.0"
+				iyy="0.01"
+				iyz="0.0"
+				izz="0.01"/>
         	</inertial>
 		</link>
@@ -79,5 +74,5 @@
 	<joint name="world_2_chassis" type='fixed'>
 		<origin xyz="0 0 0.025" rpy="0 0 0"/>
-		<parent link='base_footprint'/>
+		<parent link='world'/>
 		<child link='base_link'/>
 	</joint>
@@ -102,36 +97,33 @@
         <child link="wheel_d"/>
     </joint>
-	<ros2_control name="GazeboSimSystem" type="system">
+	<ros2_control name="GazeboSystem" type="system">
 	    <hardware>
-            <plugin>mock_components/GenericSystem</plugin>
-            <param name="mock_sensor_commands">false</param>
-            <param name="state_following_offset">0.0</param>
+            <plugin>gz_ros2_control/GazeboSimSystem</plugin>
         </hardware>
 		<joint name="chassis_to_wheel_a">
    			<command_interface name="velocity"/>
+			<state_interface name="position"/>
 			<state_interface name="velocity"/>
-   			<state_interface name="position"/>
  		</joint>
 		<joint name="chassis_to_wheel_b">
    			<command_interface name="velocity"/>
+			<state_interface name="position"/>
 			<state_interface name="velocity"/>
-   			<state_interface name="position"/>
  		</joint>
 		<joint name="chassis_to_wheel_c">
    			<command_interface name="velocity"/>
+			<state_interface name="position"/>
 			<state_interface name="velocity"/>
-   			<state_interface name="position"/>
  		</joint>
 		<joint name="chassis_to_wheel_d">
    			<command_interface name="velocity"/>
+			<state_interface name="position"/>
 			<state_interface name="velocity"/>
-   			<state_interface name="position"/>
  		</joint>
 	</ros2_control>
 	<gazebo>
-  		<plugin filename="ros2_control-system.so" name="gz_ros2_control::GazeboSimROS2ControlPlugin">
-    		<parameters>package://vex_robot/config/omni_wheel_params.yaml</parameters>
-			<controller_manager_prefix_node_name>controller_manager</controller_manager_prefix_node_name>
+  		<plugin filename="gz_ros2_control-system" name="gz_ros2_control::GazeboSimROS2ControlPlugin">
+			<parameters>$(find robot_gazebo)/config/omni_wheel_params.yaml</parameters>
   		</plugin>
 	</gazebo>
-</model>
+</robot>

Commit message: fixed frames on wheels

File: robot_gazebo/models/x_drive.urdf.xacro (robot description, xacro)
@@ -4,6 +4,9 @@
 	<xacro:property name="model_path" value="package://robot_description/models"/>
 	<xacro:property name="package_path" value="package://robot_gazebo/config"/>
+<!--
 	<xacro:property name="pi_4" value="0.7854"/>
+	<xacro:property name="pi" value="3.14159"/>
 	<xacro:property name="pi_2" value="1.5708"/>
+	<xacro:property name="pi_3/4" value="${pi_3}+${pi_4}"/> -->
 	<xacro:property name="wheel_rot" value="3.69138"/>
 	<xacro:property name="wheel_offs" value="0.14"/>
@@ -78,20 +81,20 @@
 	</joint>
 	<joint name="chassis_to_wheel_a" type="continuous">
-        <origin xyz="-${wheel_offs} ${wheel_offs} ${wheel_rad}" rpy="0 0 ${pi_4}"/>
+        <origin xyz="-${wheel_offs} ${wheel_offs} ${wheel_rad}" rpy="0 0 ${pi/4}"/>
         <parent link="base_link"/>
         <child link="wheel_a"/>
     </joint>
 	<joint name="chassis_to_wheel_b" type="continuous">
-        <origin xyz="${wheel_offs} -${wheel_offs} ${wheel_rad}" rpy="0 0 ${pi_4}"/>
+        <origin xyz="${wheel_offs} -${wheel_offs} ${wheel_rad}" rpy="0 0 ${-3* (pi/4)}"/>
         <parent link="base_link"/>
         <child link="wheel_b"/>
     </joint>
 	<joint name="chassis_to_wheel_c" type="continuous">
-        <origin xyz="${wheel_offs} ${wheel_offs} ${wheel_rad}" rpy="0 0 -${pi_4}"/>
+        <origin xyz="${wheel_offs} ${wheel_offs} ${wheel_rad}" rpy="0 0 -${pi/4}"/>
         <parent link="base_link"/>
         <child link="wheel_c"/>
     </joint>
 	<joint name="chassis_to_wheel_d" type="continuous">
-        <origin xyz="-${wheel_offs} -${wheel_offs} ${wheel_rad}" rpy="0 0 -${pi_4}"/>
+        <origin xyz="-${wheel_offs} -${wheel_offs} ${wheel_rad}" rpy="0 0 ${3 *(pi/4)}"/>
         <parent link="base_link"/>
         <child link="wheel_d"/>

Commit message: wheels now rotate correctly

File: robot_gazebo/models/x_drive.urdf.xacro (robot description, xacro)
@@ -4,12 +4,8 @@
 	<xacro:property name="model_path" value="package://robot_description/models"/>
 	<xacro:property name="package_path" value="package://robot_gazebo/config"/>
-<!--
-	<xacro:property name="pi_4" value="0.7854"/>
-	<xacro:property name="pi" value="3.14159"/>
-	<xacro:property name="pi_2" value="1.5708"/>
-	<xacro:property name="pi_3/4" value="${pi_3}+${pi_4}"/> -->
-	<xacro:property name="wheel_rot" value="3.69138"/>
+	<!-- <xacro:property name="wheel_rot" value="3.69138"/> -->
 	<xacro:property name="wheel_offs" value="0.14"/>
 	<xacro:property name="wheel_rad" value="0.01375"/>
+	<xacro:property name="wheel_width" value="0.02159"/>
 	<!--world link-->
 	<link name='world'/>
@@ -45,6 +41,8 @@
 		<link name="${name}">
 			<visual>
+			<origin xyz="0 0 0" rpy="${pi/2} 0 0"/>
 				<geometry>
-					<mesh filename='${model_path}/wheel.dae'/>
+					<!-- <mesh filename='${model_path}/wheel.dae'/> -->
+					<cylinder radius='${wheel_rad*2}' length='${wheel_width}' />
 				</geometry>
 				<material name="dark_grey">
@@ -53,6 +51,8 @@
 			</visual>
 			<collision>
+			<origin xyz="0 0 0" rpy="${pi/2} 0 0"/>
 				<geometry>
-					<mesh filename='${model_path}/wheel.dae'/>
+					<!-- <mesh filename='${model_path}/wheel.dae'/> -->
+					<cylinder radius='${wheel_rad*2}' length='${wheel_width}' />
 				</geometry>
 			</collision>
@@ -84,4 +84,5 @@
         <parent link="base_link"/>
         <child link="wheel_a"/>
+		<axis xyz="0 1 0"/>
     </joint>
 	<joint name="chassis_to_wheel_b" type="continuous">
@@ -89,4 +90,5 @@
         <parent link="base_link"/>
         <child link="wheel_b"/>
+		<axis xyz="0 1 0"/>
     </joint>
 	<joint name="chassis_to_wheel_c" type="continuous">
@@ -94,4 +96,5 @@
         <parent link="base_link"/>
         <child link="wheel_c"/>
+		<axis xyz="0 1 0"/>
     </joint>
 	<joint name="chassis_to_wheel_d" type="continuous">
@@ -99,4 +102,5 @@
         <parent link="base_link"/>
         <child link="wheel_d"/>
+		<axis xyz="0 1 0"/>
     </joint>
 	<ros2_control name="GazeboSystem" type="system">

Commit message: it moves

File: robot_gazebo/models/x_drive.urdf.xacro (robot description, xacro)
@@ -1,13 +1,13 @@
 <?xml version='1.0'?>
 <robot name="x_drive" xmlns:xacro="http://www.ros.org/wiki/xacro" xmlns:gz="http://gazebosim.org/schema">
+	<static>false</static>
 	<!-- properties-->
 	<xacro:property name="model_path" value="package://robot_description/models"/>
 	<xacro:property name="package_path" value="package://robot_gazebo/config"/>
-	<!-- <xacro:property name="wheel_rot" value="3.69138"/> -->
 	<xacro:property name="wheel_offs" value="0.14"/>
 	<xacro:property name="wheel_rad" value="0.01375"/>
 	<xacro:property name="wheel_width" value="0.02159"/>
 	<!--world link-->
-	<link name='world'/>
+	<link name='base_footprint'/>
 	<!--chassis link-->
 	<link name="base_link">
@@ -16,4 +16,7 @@
 				<mesh filename='${model_path}/chassis.dae'/>
 			</geometry>
+			<material name="pink">
+                <color rgba="0.93 0.28 0.60 1.0"/>
+			</material>
 		</visual>
 		<collision>
@@ -21,7 +24,13 @@
 				<mesh filename='${model_path}/chassis.dae'/>
 			</geometry>
-			<material name="pink">
-				<color rgba="237 72 154 1.0"/>
-			</material>
+			<surface>
+                    <friction>
+                        <ode>
+                            <mu>1.0</mu>
+                            <mu2>1.0</mu2>
+                            <fdir1>0 0 1</fdir1>
+                        </ode>
+                    </friction>
+                </surface>
 		</collision>
 		<inertial>
@@ -74,8 +83,8 @@
 	<xacro:wheel_link name="wheel_c"/>
 	<xacro:wheel_link name="wheel_d"/>
-	<!-- joints-->
+	<!-- joints -->
 	<joint name="world_2_chassis" type='fixed'>
 		<origin xyz="0 0 0.025" rpy="0 0 0"/>
-		<parent link='world'/>
+		<parent link='base_footprint'/>
 		<child link='base_link'/>
 	</joint>

Commit message: fixed inertia problems

File: robot_gazebo/models/x_drive.urdf.xacro (robot description, xacro)
@@ -9,5 +9,17 @@
 	<xacro:property name="wheel_width" value="0.02159"/>
 	<!--world link-->
-	<link name='base_footprint'/>
+	<link name='base_footprint'>
+	 <!-- <inertial>
+            <origin xyz="0 0 0" rpy="0 0 0"/>
+            <mass value="0.01"/>
+            <inertia
+                ixx="0.001"
+                ixy="0.0"
+                ixz="0.0"
+                iyy="0.001"
+                iyz="0.0"
+                izz="0.001"/>
+        </inertial> -->
+	</link>
 	<!--chassis link-->
 	<link name="base_link">
@@ -27,12 +39,12 @@
 		<inertial>
             <origin xyz="0 0 0" rpy="0 0 0"/>
-            <mass value="8.789"/>
+            <mass value="4.54"/>
            <inertia
-      			ixx="0.01"
+      			ixx="0.05487"
 				ixy="0.0"
 				ixz="0.0"
-				iyy="0.01"
+				iyy="0.05487"
 				iyz="0.0"
-				izz="0.01"/>
+				izz="0.10974"/>
     		</inertial>
 	</link>
@@ -68,12 +80,12 @@
 			<inertial>
             	<origin xyz="0 0 0" rpy="0 0 0"/>
-            	<mass value="0.076"/>
+            	<mass value="0.070"/>
 				<inertia
-      			ixx="0.01"
+      			ixx="0.001"
 				ixy="0.0"
 				ixz="0.0"
-				iyy="0.01"
+				iyy="0.001"
 				iyz="0.0"
-				izz="0.01"/>
+				izz="0.001"/>
         	</inertial>
 		</link>

Commit message: fixed most comments

File: robot_gazebo/models/x_drive.urdf.xacro (robot description, xacro)
@@ -9,17 +9,5 @@
 	<xacro:property name="wheel_width" value="0.02159"/>
 	<!--world link-->
-	<link name='base_footprint'>
-	 <!-- <inertial>
-            <origin xyz="0 0 0" rpy="0 0 0"/>
-            <mass value="0.01"/>
-            <inertia
-                ixx="0.001"
-                ixy="0.0"
-                ixz="0.0"
-                iyy="0.001"
-                iyz="0.0"
-                izz="0.001"/>
-        </inertial> -->
-	</link>
+	<link name='base_footprint'/>
 	<!--chassis link-->
 	<link name="base_link">
@@ -55,5 +43,4 @@
 			<origin xyz="0 0 0" rpy="${pi/2} 0 0"/>
 				<geometry>
-					<!-- <mesh filename='${model_path}/wheel.dae'/> -->
 					<cylinder radius='${wheel_rad*2}' length='${wheel_width}' />
 				</geometry>
@@ -65,5 +52,4 @@
 			<origin xyz="0 0 0" rpy="${pi/2} 0 0"/>
 				<geometry>
-					<!-- <mesh filename='${model_path}/wheel.dae'/> -->
 					<cylinder radius='${wheel_rad*2}' length='${wheel_width}' />
 				</geometry>
@@ -125,4 +111,5 @@
 		<axis xyz="0 1 0"/>
     </joint>
+	<!-- ROS 2 Control-->
 	<ros2_control name="GazeboSystem" type="system">
 	    <hardware>
@@ -150,4 +137,5 @@
  		</joint>
 	</ros2_control>
+	<!-- gazebo stuff -->
 	<gazebo>
   		<plugin filename="gz_ros2_control-system" name="gz_ros2_control::GazeboSimROS2ControlPlugin">
