Commit message: robot.launch.py did not crash

File: robot_description/urdf/x_drive.urdf.xacro (robot description, xacro)
@@ -13,12 +13,7 @@
     <link name="base_link">
         <visual>
-            <!--
+            <origin xyz="0 0 0.05" rpy="0 0 0"/>
             <geometry>
-                <mesh filename='${model_path}/chassis-v2.dae'/>
-            </geometry>
-            -->
-            <origin xyz="0 0 0.25" rpy="0 0 0"/>
-            <geometry>
-                <cylinder length="0.0315" radius="0.055"/>
+                <box size='0.20 0.20 0.02'/>
             </geometry>
             <material name="pink">
@@ -27,12 +22,7 @@
         </visual>
         <collision>
-            <!--
+            <origin xyz="0 0 0.05" rpy="0 0 0"/>
             <geometry>
-                <mesh filename='${model_path}/chassis.dae'/>
-            </geometry>
-            -->
-            <origin xyz="0 0 0.25" rpy="0 0 0"/>
-            <geometry>
-                <cylinder length="0.0315" radius="0.055"/>
+                 <box size='0.20 0.20 0.02'/>
             </geometry>
         </collision>
@@ -41,5 +31,5 @@
             <mass value="4.54"/>
            <inertia
-                  ixx="0.05487"
+                ixx="0.05487"
                 ixy="0.0"
                 ixz="0.0"
@@ -51,32 +41,4 @@
     <!--Sensor links-->
     <link name="imu_link"/>
-    <link name="laser_frame">
-            <visual>
-                <origin xyz="0 0 0.0" rpy="0 0 0"/>
-                <geometry>
-                    <cylinder length="0.0315" radius="0.055"/>
-                </geometry>
-                <material name="dark_grey">
-                    <color rgba="0.2 0.2 0.2 1.0"/>
-                </material>
-            </visual>
-            <collision>
-                <origin xyz="0.015 0 -0.0065" rpy="0 0 0"/>
-                <geometry>
-                    <cylinder length="0.0315" radius="0.055"/>
-                </geometry>
-            </collision>
-            <inertial>
-                <origin xyz="0 0 0" />
-                <mass value="0.114" />
-                <inertia
-                ixx="0.001"
-                ixy="0.0"
-                ixz="0.0"
-                iyy="0.001"
-                iyz="0.0"
-                izz="0.001"/>
-            </inertial>
-    </link>
     <!-- wheels -->
     <xacro:macro name="wheel_link" params="name">
@@ -109,12 +71,4 @@
             </inertial>
         </link>
-    <gazebo reference="${name}">
-        <mu1 value="0.2"/>
-        <mu2 value="1.5"/>
-        <kp value="10000000.0" />
-        <kd value="10000.0" />
-        <fdir1 value="0 0 1"/>
-        <maxContacts value= "1"/>
-    </gazebo>
     </xacro:macro>
     <xacro:wheel_link name="wheel_a"/>
@@ -158,9 +112,43 @@
         <origin xyz="0 0 0.04" rpy="0 0 0"/>
     </joint>
-    <joint name="laser_joint" type="fixed">
-         <parent link="base_link"/>
-         <child link="laser_frame"/>
-        <origin xyz="0 0 0.2" rpy="0 0 0"/>
-     </joint>
+    <xacro:macro name='TiMXXS_lidar' params='sensor_number xyz yaw'>
+        <!-- lidar link -->
+        <link name="laser_frame_${sensor_number}"> <!-- make sure TiM7xxS has the same frame ID in the lidar launch file!-->
+            <visual>
+                <origin xyz="0 0 0.0" rpy="0 0 0"/>
+                <geometry>
+                    <cylinder length="0.02" radius="0.02"/>
+                </geometry>
+                <material name="dark_grey">
+                    <color rgba="0.2 0.2 0.2 1.0"/>
+                </material>
+            </visual>
+            <collision>
+                <origin xyz="0 0 0" rpy="0 0 0"/>
+                <geometry>
+                    <cylinder length="0.02" radius="0.02"/>
+                </geometry>
+            </collision>
+            <inertial>
+                <origin xyz="0 0 0" />
+                <mass value="0.114" />
+                <inertia
+                ixx="0.001"
+                ixy="0.0"
+                ixz="0.0"
+                iyy="0.001"
+                iyz="0.0"
+                izz="0.001"/>
+            </inertial>
+        </link>
+        <!-- lidar joint -->
+        <joint name="laser_joint_${sensor_number}" type="fixed">
+            <parent link="base_link"/>
+            <child link="laser_frame_${sensor_number}"/>
+            <origin xyz="${xyz}" rpy="0 0 ${yaw}"/>
+        </joint>
+    </xacro:macro>
+    <xacro:TiMXXS_lidar sensor_number='1' xyz="0.13 0.12 0.14" yaw='-${pi/4}'/>
+    <xacro:TiMXXS_lidar sensor_number='2' xyz="-0.13 0.12 0.14" yaw='${pi/4}'/>
     <!-- ROS 2 Control-->
     <ros2_control name="GazeboSystem" type="system">
@@ -191,40 +179,3 @@
          </joint>
     </ros2_control>
-    <!-- Gazebo Sim Plugins -->
-    <gazebo>
-          <plugin filename="gz_ros2_control-system" name="gz_ros2_control::GazeboSimROS2ControlPlugin">
-            <parameters>$(find robot_gazebo)/config/omni_wheel_params.yaml</parameters>
-          </plugin>
-    </gazebo>
-    <!-- Sensor Gazebo Tag-->
-    <gazebo reference="laser_frame">
-        <sensor name="lidar" type="gpu_lidar">
-            <pose>0 0 0 0 0 0</pose>
-            <always_on>true</always_on>
-            <visualize>true</visualize>
-            <update_rate>10</update_rate>
-            <topic>scan</topic>
-            <gz_frame_id>laser_frame</gz_frame_id>
-            <lidar>
-                <scan>
-                    <horizontal>
-                        <samples>720</samples>
-                        <resolution>1</resolution>
-                        <min_angle>-3.14</min_angle>
-                        <max_angle>3.14</max_angle>
-                    </horizontal>
-                </scan>
-                <range>
-                    <min>0.05</min>
-                    <max>10.0</max>
-                    <resolution>0.01</resolution>
-                </range>
-                <noise>
-                    <type>gaussian</type>
-                    <mean>0.0</mean>
-                    <stddev>0.01</stddev>
-                </noise>
-            </lidar>
-        </sensor>
-    </gazebo>
 </robot>

Commit message: dual lidar in correct frame

File: robot_description/urdf/x_drive.urdf.xacro (robot description, xacro)
@@ -5,7 +5,12 @@
     <xacro:property name="model_path" value="package://robot_description/models"/>
     <xacro:property name="package_path" value="package://robot_gazebo/config"/>
+    <!--Wheel properties-->
     <xacro:property name="wheel_offs" value="0.14"/>
     <xacro:property name="wheel_rad" value="0.0349253"/>
     <xacro:property name="wheel_width" value="0.02159"/>
+    <!-- Camera properties-->
+    <xacro:property name="camera_x" value="0.114"/>
+    <xacro:property name="camera_y" value="0.116"/>
+    <xacro:property name="camera_z" value="0.197"/>
     <!--world link-->
     <link name='base_footprint'/>
@@ -13,4 +18,9 @@
     <link name="base_link">
         <visual>
+            <!--
+            <geometry>
+                <mesh filename='${model_path}/chassis-v2.dae'/>
+            </geometry>
+            -->
             <origin xyz="0 0 0.05" rpy="0 0 0"/>
             <geometry>
@@ -22,4 +32,9 @@
         </visual>
         <collision>
+            <!--
+            <geometry>
+                <mesh filename='${model_path}/chassis.dae'/>
+            </geometry>
+            -->
             <origin xyz="0 0 0.05" rpy="0 0 0"/>
             <geometry>
@@ -39,5 +54,5 @@
             </inertial>
     </link>
-    <!--Sensor links-->
+    <!--imu link-->
     <link name="imu_link"/>
     <!-- wheels -->
@@ -71,4 +86,12 @@
             </inertial>
         </link>
+        <gazebo reference="${name}">
+            <mu1 value="0.2"/>
+            <mu2 value="1.5"/>
+            <kp value="10000000.0" />
+            <kd value="10000.0" />
+            <fdir1 value="0 0 1"/>
+            <maxContacts value= "1"/>
+        </gazebo>
     </xacro:macro>
     <xacro:wheel_link name="wheel_a"/>
@@ -76,43 +99,78 @@
     <xacro:wheel_link name="wheel_c"/>
     <xacro:wheel_link name="wheel_d"/>
-    <!-- joints -->
-    <joint name="footprint_2_link" type='fixed'>
-        <origin xyz="0 0 0.025" rpy="0 0 0"/>
-        <parent link='base_footprint'/>
-        <child link='base_link'/>
-    </joint>
-    <joint name="chassis_to_wheel_a" type="continuous">
-        <origin xyz="-${wheel_offs} ${wheel_offs} ${wheel_rad}" rpy="0 0 ${pi/4}"/>
-        <parent link="base_link"/>
-        <child link="wheel_a"/>
-        <axis xyz="0 1 0"/>
-    </joint>
-    <joint name="chassis_to_wheel_b" type="continuous">
-        <origin xyz="${wheel_offs} -${wheel_offs} ${wheel_rad}" rpy="0 0 ${-3* (pi/4)}"/>
-        <parent link="base_link"/>
-        <child link="wheel_b"/>
-        <axis xyz="0 1 0"/>
-    </joint>
-    <joint name="chassis_to_wheel_c" type="continuous">
-        <origin xyz="${wheel_offs} ${wheel_offs} ${wheel_rad}" rpy="0 0 -${pi/4}"/>
-        <parent link="base_link"/>
-        <child link="wheel_c"/>
-        <axis xyz="0 1 0"/>
-    </joint>
-    <joint name="chassis_to_wheel_d" type="continuous">
-        <origin xyz="-${wheel_offs} -${wheel_offs} ${wheel_rad}" rpy="0 0 ${3 *(pi/4)}"/>
-        <parent link="base_link"/>
-        <child link="wheel_d"/>
-        <axis xyz="0 1 0"/>
-    </joint>
-    <!--Sensor Joints-->
-    <joint name="imu_joint" type="fixed">
-        <parent link="base_link"/>
-        <child link="imu_link"/>
-        <origin xyz="0 0 0.04" rpy="0 0 0"/>
-    </joint>
+    <!-- USB Camera x4 -->
+    <xacro:macro name='usb_cam' params='camera_name xyz rpy'>
+        <link name='${camera_name}_link'>
+            <visual>
+                <geometry>
+                    <box size='0.02 0.02 0.02'/>
+                </geometry>
+                <material name="dark_grey">
+                    <color rgba="0.2 0.2 0.2 1.0"/>
+                </material>
+            </visual>
+            <collision>
+                <geometry>
+                    <box size='0.02 0.02 0.02'/>
+                </geometry>
+                <material name="dark_grey">
+                    <color rgba="0.2 0.2 0.2 1.0"/>
+                </material>
+            </collision>
+            <inertial>
+                <origin xyz="0 0 0" rpy="0 0 0"/>
+                <mass value="0.01"/>
+                <inertia
+                    ixx="0.000001"
+                    ixy="0.0"
+                    ixz="0.0"
+                    iyy="0.000001"
+                    iyz="0.0"
+                    izz="0.000001"/>
+            </inertial>
+        </link>
+        <joint name="${camera_name}_joint" type="fixed">
+            <parent link="base_link"/>
+            <child link="${camera_name}_link"/>
+            <origin xyz="${xyz}" rpy="${rpy}"/>
+        </joint>
+        <link name="${camera_name}_link_optical"/>
+        <joint name="${camera_name}_optical_joint" type="fixed">
+            <parent link="${camera_name}_link"/>
+            <child link="${camera_name}_link_optical"/>
+            <origin xyz="0 0 0" rpy="-1.5708 0 -1.5708"/>
+        </joint>
+        <gazebo reference='${camera_name}_link'>
+            <sensor name='${camera_name}_sensor' type="camera">
+                <pose>0 0 0 0 0 0</pose>
+                <camera>
+                    <horizontal_fov>1.26</horizontal_fov>
+                    <image>
+                        <width>1920</width>
+                        <height>1200</height>
+                        <format>R8G8B8</format>
+                    </image>
+                    <clip>
+                        <near>0.001</near>
+                        <far>20</far>
+                    </clip>
+                </camera>
+                <always_on>true</always_on>
+                <update_rate>10</update_rate> <!-- i think our cameras run at 90fps max, but for sim, even 30 kills it. maybe 10 will be better? -->
+                <visualize>true</visualize>
+                <topic>/${camera_name}/image_raw</topic>
+                <gz_frame_id>${camera_name}_link_optical</gz_frame_id>
+            </sensor>
+        </gazebo>
+    </xacro:macro>
+    <!-- make sure to update ROS bridge in spawn_robot.launch.py! -->
+    <xacro:usb_cam camera_name='cam1' xyz='-${camera_x} ${camera_y} ${camera_z}' rpy='0 0 ${3*pi/4}'/>
+    <xacro:usb_cam camera_name='cam2' xyz='-${camera_x} -${camera_y} ${camera_z}' rpy='0 0 -${3*pi/4}'/>
+    <xacro:usb_cam camera_name='cam3' xyz='${camera_x} ${camera_y} ${camera_z}' rpy='0 0 ${pi/4}'/>
+    <xacro:usb_cam camera_name='cam4' xyz='${camera_x} -${camera_y} ${camera_z}' rpy='0 0 -${pi/4}'/>
+    <!-- LiDAR x2 -->
     <xacro:macro name='TiMXXS_lidar' params='sensor_number xyz yaw'>
         <!-- lidar link -->
-        <link name="laser_frame_${sensor_number}"> <!-- make sure TiM7xxS has the same frame ID in the lidar launch file!-->
+        <link name="laser_frame_${sensor_number}">
             <visual>
                 <origin xyz="0 0 0.0" rpy="0 0 0"/>
@@ -148,7 +206,74 @@
             <origin xyz="${xyz}" rpy="0 0 ${yaw}"/>
         </joint>
+        <!-- actual sensor-->
+        <gazebo reference="laser_frame_${sensor_number}">
+            <sensor name="lidar_${sensor_number}" type="gpu_lidar">
+                <pose>0 0 0 0 0 0</pose>
+                <always_on>true</always_on>
+                <visualize>true</visualize>
+                <update_rate>10</update_rate>
+                <topic>scan_${sensor_number}</topic>
+                <gz_frame_id>laser_frame_${sensor_number}</gz_frame_id>
+                <lidar>
+                    <scan>
+                        <horizontal>
+                            <samples>720</samples>
+                            <resolution>1</resolution>
+                            <min_angle>-0.785398163</min_angle>
+                            <max_angle>3.92699</max_angle>
+                        </horizontal>
+                    </scan>
+                    <range>
+                        <min>0.15</min>
+                        <max>10.0</max>
+                        <resolution>0.01</resolution>
+                    </range>
+                    <noise>
+                        <type>gaussian</type>
+                        <mean>0.0</mean>
+                        <stddev>0.01</stddev>
+                    </noise>
+                </lidar>
+            </sensor>
+        </gazebo>
     </xacro:macro>
     <xacro:TiMXXS_lidar sensor_number='1' xyz="0.13 0.12 0.14" yaw='-${pi/4}'/>
     <xacro:TiMXXS_lidar sensor_number='2' xyz="-0.13 0.12 0.14" yaw='${pi/4}'/>
+    <!-- Joints -->
+    <joint name="footprint_2_link" type='fixed'>
+        <origin xyz="0 0 0.025" rpy="0 0 0"/>
+        <parent link='base_footprint'/>
+        <child link='base_link'/>
+    </joint>
+    <joint name="chassis_to_wheel_a" type="continuous">
+        <origin xyz="-${wheel_offs} ${wheel_offs} ${wheel_rad}" rpy="0 0 ${pi/4}"/>
+        <parent link="base_link"/>
+        <child link="wheel_a"/>
+        <axis xyz="0 1 0"/>
+    </joint>
+    <joint name="chassis_to_wheel_b" type="continuous">
+        <origin xyz="${wheel_offs} -${wheel_offs} ${wheel_rad}" rpy="0 0 ${-3* (pi/4)}"/>
+        <parent link="base_link"/>
+        <child link="wheel_b"/>
+        <axis xyz="0 1 0"/>
+    </joint>
+    <joint name="chassis_to_wheel_c" type="continuous">
+        <origin xyz="${wheel_offs} ${wheel_offs} ${wheel_rad}" rpy="0 0 -${pi/4}"/>
+        <parent link="base_link"/>
+        <child link="wheel_c"/>
+        <axis xyz="0 1 0"/>
+    </joint>
+    <joint name="chassis_to_wheel_d" type="continuous">
+        <origin xyz="-${wheel_offs} -${wheel_offs} ${wheel_rad}" rpy="0 0 ${3 *(pi/4)}"/>
+        <parent link="base_link"/>
+        <child link="wheel_d"/>
+        <axis xyz="0 1 0"/>
+    </joint>
+    <!--Sensor Joints-->
+    <joint name="imu_joint" type="fixed">
+        <parent link="base_link"/>
+        <child link="imu_link"/>
+        <origin xyz="0 0 0.04" rpy="0 0 0"/>
+    </joint>
     <!-- ROS 2 Control-->
     <ros2_control name="GazeboSystem" type="system">

Commit message: removed sim stuff from urdf

File: robot_description/urdf/x_drive.urdf.xacro (robot description, xacro)
@@ -1,5 +1,6 @@
 <?xml version='1.0'?>
-<robot name="x_drive" xmlns:xacro="http://www.ros.org/wiki/xacro" xmlns:gz="http://gazebosim.org/schema">
+<robot name="x_drive" xmlns:xacro="http://www.ros.org/wiki/xacro">
     <static>false</static>
+    <xacro:include filename="$(find robot_description)/urdf/robot_variables.xacro"/>
     <!-- properties-->
     <xacro:property name="model_path" value="package://robot_description/models"/>
@@ -18,9 +19,4 @@
     <link name="base_link">
         <visual>
-            <!--
-            <geometry>
-                <mesh filename='${model_path}/chassis-v2.dae'/>
-            </geometry>
-            -->
             <origin xyz="0 0 0.05" rpy="0 0 0"/>
             <geometry>
@@ -32,9 +28,4 @@
         </visual>
         <collision>
-            <!--
-            <geometry>
-                <mesh filename='${model_path}/chassis.dae'/>
-            </geometry>
-            -->
             <origin xyz="0 0 0.05" rpy="0 0 0"/>
             <geometry>
@@ -141,26 +132,4 @@
             <origin xyz="0 0 0" rpy="-1.5708 0 -1.5708"/>
         </joint>
-        <gazebo reference='${camera_name}_link'>
-            <sensor name='${camera_name}_sensor' type="camera">
-                <pose>0 0 0 0 0 0</pose>
-                <camera>
-                    <horizontal_fov>1.26</horizontal_fov>
-                    <image>
-                        <width>1920</width>
-                        <height>1200</height>
-                        <format>R8G8B8</format>
-                    </image>
-                    <clip>
-                        <near>0.001</near>
-                        <far>20</far>
-                    </clip>
-                </camera>
-                <always_on>true</always_on>
-                <update_rate>10</update_rate> <!-- i think our cameras run at 90fps max, but for sim, even 30 kills it. maybe 10 will be better? -->
-                <visualize>true</visualize>
-                <topic>/${camera_name}/image_raw</topic>
-                <gz_frame_id>${camera_name}_link_optical</gz_frame_id>
-            </sensor>
-        </gazebo>
     </xacro:macro>
     <!-- make sure to update ROS bridge in spawn_robot.launch.py! -->
@@ -206,38 +175,7 @@
             <origin xyz="${xyz}" rpy="0 0 ${yaw}"/>
         </joint>
-        <!-- actual sensor-->
-        <gazebo reference="laser_frame_${sensor_number}">
-            <sensor name="lidar_${sensor_number}" type="gpu_lidar">
-                <pose>0 0 0 0 0 0</pose>
-                <always_on>true</always_on>
-                <visualize>true</visualize>
-                <update_rate>10</update_rate>
-                <topic>scan_${sensor_number}</topic>
-                <gz_frame_id>laser_frame_${sensor_number}</gz_frame_id>
-                <lidar>
-                    <scan>
-                        <horizontal>
-                            <samples>720</samples>
-                            <resolution>1</resolution>
-                            <min_angle>-0.785398163</min_angle>
-                            <max_angle>3.92699</max_angle>
-                        </horizontal>
-                    </scan>
-                    <range>
-                        <min>0.15</min>
-                        <max>10.0</max>
-                        <resolution>0.01</resolution>
-                    </range>
-                    <noise>
-                        <type>gaussian</type>
-                        <mean>0.0</mean>
-                        <stddev>0.01</stddev>
-                    </noise>
-                </lidar>
-            </sensor>
-        </gazebo>
     </xacro:macro>
-    <xacro:TiMXXS_lidar sensor_number='1' xyz="0.13 0.12 0.14" yaw='-${pi/4}'/>
-    <xacro:TiMXXS_lidar sensor_number='2' xyz="-0.13 0.12 0.14" yaw='${pi/4}'/>
+    <xacro:TiMXXS_lidar sensor_number='1' xyz="-0.13 0.12 0.14" yaw='${3* pi/4}'/>
+    <xacro:TiMXXS_lidar sensor_number='2' xyz="-0.13 -0.12 0.14" yaw='-${ 3* pi/4}'/>
     <!-- Joints -->
     <joint name="footprint_2_link" type='fixed'>
@@ -277,5 +215,5 @@
     </joint>
     <!-- ROS 2 Control-->
-    <ros2_control name="GazeboSystem" type="system">
+    <ros2_control name="DriveSystem" type="system">
         <hardware>
             <plugin>mock_components/GenericSystem</plugin>

Commit message: confirmed lidar launch works on hw

File: robot_description/urdf/x_drive.urdf.xacro (robot description, xacro)
@@ -45,4 +45,32 @@
             </inertial>
     </link>
+    <link name="intake_link">
+        <visual>
+            <origin xyz='0 0 0' rpy='0 0 0'/>
+            <geometry>
+                <box size='0.189 0.146 0.20'/>
+            </geometry>
+            <material name="light-blue">
+                <color rgba="0.68 0.85 0.9 1"/>
+            </material>
+        </visual>
+        <collision>
+            <origin xyz="0 0 0" rpy="0 0 0"/>
+            <geometry>
+                <box size='0.189 0.146 0.10'/>
+            </geometry>
+        </collision>
+        <inertial>
+            <origin xyz="0 0 0" rpy="0 0 0"/>
+            <mass value="0.070"/>
+            <inertia
+            ixx="0.001"
+            ixy="0.0"
+            ixz="0.0"
+            iyy="0.001"
+            iyz="0.0"
+            izz="0.001"/>
+        </inertial>
+    </link>
     <!--imu link-->
     <link name="imu_link"/>
@@ -184,4 +212,9 @@
         <child link='base_link'/>
     </joint>
+    <joint name="base_2_intake" type='fixed'>
+        <origin xyz="0.0945 0 0.16" rpy="0 0 0"/>
+        <parent link='base_link'/>
+        <child link='intake_link'/>
+    </joint>
     <joint name="chassis_to_wheel_a" type="continuous">
         <origin xyz="-${wheel_offs} ${wheel_offs} ${wheel_rad}" rpy="0 0 ${pi/4}"/>

Commit message: lidar + controllers can be brought up

File: robot_description/urdf/x_drive.urdf.xacro (robot description, xacro)
@@ -5,5 +5,5 @@
     <!-- properties-->
     <xacro:property name="model_path" value="package://robot_description/models"/>
-    <xacro:property name="package_path" value="package://robot_gazebo/config"/>
+    <xacro:property name="package_path" value="package://robot_description/config"/>
     <!--Wheel properties-->
     <xacro:property name="wheel_offs" value="0.14"/>
